File: v2/v2.0.0.0/rev-/pga103_v2.0.0.0.kicad_sch (KiCad schematic)
At the start: 29 parts, among them J1 RF_IN, J2 RF_OUT, J3 RFShield_TwoPieces, U1 SPX3819M5-L-5-0, U2 PGA-103

Commit message: added pdf of schematic, board population checklist, fixed typo in V2.0.0.0 title
Other:
- title: PGA-103+ Preamplifier, Version 2.1.0.0 -> PGA-103+ Preamplifier, Version 2.0.0.0
Changed lines of the file:
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@@
   (paper "A")
   (title_block
-    (title "PGA-103+ Preamplifier, Version 2.1.0.0")
+    (title "PGA-103+ Preamplifier, Version 2.0.0.0")
     (date "2023-10-02")
     (rev "-")
